Commit message: update robot petra

File: petra_robot/urdf/petra_robot.urdf (robot description, URDF)
Before this commit: robot petra_robot, 7 links, 6 joints
Links:
- added link camera_link, mass 0.1; collision box size=.03 .03 .03; visual box size=.03 .03 .03
- added link camera_link_optical
Joints:
- added joint camera_joint: type fixed, parent base_link, child camera_link, origin xyz=0.2 0 0.05 rpy=0 0 0, axis 0 1 0
- added joint camera_optical_joint: type fixed, parent camera_link, child camera_link_optical, origin xyz=0 0 0 rpy=-1.5707 0 -1.5707

Commit message: update petra robot with new world

File: petra_robot/urdf/petra_robot.urdf (robot description, URDF)
Before this commit: robot petra_robot, 9 links, 8 joints
Links:
- link lidar_link: mass 0.5 -> 1e-5

Commit message: update petra robot

File: petra_robot/urdf/petra_robot.urdf (robot description, URDF)
Before this commit: robot petra_robot, 9 links, 8 joints
Links:
- removed link caster_wheel_link
- removed link lidar_base_link
- removed link lidar_link
- added link imu_link
- added link scan_link, mass 1e-5; collision box size=.1 .1 .1; visual mesh filename=package://petra_robot/meshes/lidar.dae
- link base_link: mass 2.0 -> 15.0; geometry collision box size=.4 .2 .1; collision sphere radius=0.0499
- link left_wheel: mass 1.0 -> 5.0; geometry collision cylinder length=.05 radius=.1; visual mesh filename=package://petra_robot/meshes/wheel.dae
- link right_wheel: mass 1.0 -> 5.0; geometry collision cylinder length=.05 radius=.1; visual mesh filename=package://petra_robot/meshes/wheel.dae
Joints:
- removed joint caster_wheel_joint
- removed joint lidar_base_joint
- removed joint lidar_joint
- added joint imu_joint: type fixed, parent base_link, child imu_link, origin xyz=0 0 0 rpy=0 0 0
- added joint scan_joint: type fixed, parent base_link, child scan_link, origin xyz=0.0 0 0.15 rpy=0 0 0, axis 0 1 0
- joint base_footprint_joint: origin xyz=0.0 0.0 0.0 rpy=0 0 0 -> xyz=0 0 0 rpy=0 0 0
- joint camera_joint: origin xyz=0.2 0 0.05 rpy=0 0 0 -> xyz=0.225 0 0.075 rpy=0 0 0
- joint left_wheel_joint: axis 0 0 1 -> 0 1 0; limit (none) -> effort=100 velocity=10; origin xyz=0.1 0.175 0.0 rpy=0 1.5708 1.5708 -> xyz=0 0.15 0 rpy=0 0 0
- joint right_wheel_joint: axis 0 0 1 -> 0 1 0; limit (none) -> effort=100 velocity=10; origin xyz=0.1 -0.175 0.00 rpy=0 1.5708 1.5708 -> xyz=0 -0.15 0 rpy=0 0 0
