Commit message: orginze petra_robot pkg

File: petra_robot/urdf/petra_robot_v1.urdf (robot description, URDF)
Before this commit: robot petra_robot, 8 links, 7 joints
Links:
- added link caster_wheel_link, mass 0.5; collision sphere radius=0.02; visual sphere radius=0.02
- link base_link: geometry collision box size=0.4 0.3 0.08; visual box size=0.4 0.3 0.08
Joints:
- added joint caster_wheel_joint: type continuous, parent base_link, child caster_wheel_link, origin xyz=-0.1 0.0 -0.06 rpy=0.0 0.0 0.0, axis 0 0 1
